File: Board/Board.kicad_sch (KiCad schematic)
At the start: 49 parts, among them J1 Conn_01x03, U1 USB-C, U13 ESP32-C6-MINI-1-N4, U3 AHT20, U4 Tactile-Switch, U6 Light sensor, U7 Tactile-Switch, U8 Slide-Switch, U9 Battery-Spring

Commit message: Update and fix Board and Panel
Parts:
- U1: JLCPCB Position Offset (none) -> 0,0.83,0
- U3: JLCPCB Rotation Offset (none) -> 180
- U8: JLCPCB Position Offset 0,0,-0.5 -> (none)
Changed lines of the file:
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@@
 			)
 		)
-		(property "JLCPCB Position Offset" "0,0,-0.5"
+		(property "JLCPCB Position Offset" ""
 			(at 118.745 128.27 0)
 			(effects
@@
 			)
 		)
+		(property "JLCPCB Position Offset" "0,0.83,0"
+			(at 163.195 180.975 0)
+			(effects
+				(font
+					(size 1.27 1.27)
+				)
+				(hide yes)
+			)
+		)
 		(pin "A7"
 		)
@@
 			(at 33.02 91.44 0)
 			(effects
+				(font
+					(size 1.27 1.27)
+				)
+				(hide yes)
+			)
+		)
+		(property "JLCPCB Rotation Offset" "180"
+			(at 33.02 91.44 0)
+			(effects

Commit message: Add missing tabs to blumy panel
Parts:
- added U14, U5: ~, CustomFootprints:MouseBites5mm, symbol Custom_Parts:MouseBite5mm
Changed lines of the file:
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@@
+	)
+	(symbol
+		(lib_id "Custom_Parts:MouseBite5mm")
+		(at 219.71 163.83 0)
+		(unit 1)
+		(exclude_from_sim no)
+		(in_bom no)
+		(on_board yes)
+		(dnp yes)
+		(fields_autoplaced yes)
+		(property "Reference" "U5"
+			(at 219.71 162.56 0)
+			(effects
+				(font
+					(size 1.27 1.27)
+				)
+			)
+		)
+		(property "Value" "~"
+			(at 219.71 163.83 0)
+			(effects
+				(font
+					(size 1.27 1.27)
+				)
+			)
+		)
+		(property "Footprint" "CustomFootprints:MouseBites5mm"
+			(at 219.71 163.83 0)
+			(effects
+				(font
+					(size 1.27 1.27)
+				)
+				(hide yes)
+			)
+		)
+		(property "Datasheet" ""
+			(at 219.71 163.83 0)
+			(effects
+				(font
+					(size 1.27 1.27)
+				)
+				(hide yes)
+			)
+		)
+		(property "Description" ""
+			(at 219.71 163.83 0)
+			(effects
+				(font
+					(size 1.27 1.27)
+				)
+				(hide yes)
+			)
+		)
+		(property "MPN" "/"
+			(at 219.71 163.83 0)
+			(effects
+				(font
+					(size 1.27 1.27)
+				)
+				(hide yes)
+			)
+		)
+		(instances
+			(project "Board"
+				(path "/fa2a81f8-bf39-4c28-beef-a6fc807c4564"
+					(reference "U5")
+					(unit 1)
+				)
+			)
+		)
 	)
 	(symbol
@@
 					(unit 1)
 				)
+			)
+		)
+	)
+	(symbol
+		(lib_id "Custom_Parts:MouseBite5mm")
+		(at 231.14 163.83 0)
+		(unit 1)
+		(exclude_from_sim no)
+		(in_bom no)
+		(on_board yes)
+		(dnp yes)
+		(fields_autoplaced yes)
+		(property "Reference" "U14"
+			(at 231.14 162.56 0)
+			(effects
+				(font
+					(size 1.27 1.27)
+				)
+			)
+		)
+		(property "Value" "~"
+			(at 231.14 163.83 0)
+			(effects
+				(font
+					(size 1.27 1.27)
+				)
+			)
+		)
+		(property "Footprint" "CustomFootprints:MouseBites5mm"
+			(at 231.14 163.83 0)
+			(effects
+				(font
+					(size 1.27 1.27)
+				)
+				(hide yes)
+			)
+		)
+		(property "Datasheet" ""
+			(at 231.14 163.83 0)
+			(effects
+				(font
+					(size 1.27 1.27)
+				)
+				(hide yes)
+			)
+		)
+		(property "Description" ""
+			(at 231.14 163.83 0)
+			(effects
+				(font
+					(size 1.27 1.27)
+				)
+				(hide yes)
+			)
+		)
+		(property "MPN" "/"
+			(at 231.14 163.83 0)
+			(effects
+				(font
+					(size 1.27 1.27)
+				)
+				(hide yes)
+			)
+		)
+		(instances
+			(project "Board"
+				(path "/fa2a81f8-bf39-4c28-beef-a6fc807c4564"
+					(reference "U14")
+					(unit 1)
+				)

Commit message: Remove boot capacitor from blumy and flip usb bat text
Parts:
- removed C5: 100nF-Ceramic, Capacitor_SMD:C_0402_1005Metric, symbol Device:C
Changed lines of the file:
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@@
 	)
 	(junction
-		(at 254.635 99.06)
-		(diameter 0)
-		(color 0 0 0 0)
-	)
-	(junction
 		(at 205.74 101.6)
 		(diameter 0)
@@
 	)
 	(junction
-		(at 271.145 99.06)
-		(diameter 0)
-		(color 0 0 0 0)
-	)
-	(junction
 		(at 50.8 168.275)
 		(diameter 0)
@@
 	(wire
 		(pts
-			(xy 271.145 102.87) (xy 271.145 99.06)
-		)
-		(stroke
-			(width 0)
-			(type default)
-		)
-	)
-	(wire
-		(pts
 			(xy 205.74 99.06) (xy 205.74 101.6)
 		)
@@
 	(wire
 		(pts
-			(xy 254.635 99.06) (xy 255.27 99.06)
+			(xy 251.46 99.06) (xy 255.27 99.06)
 		)
 		(stroke
@@
 	(wire
 		(pts
-			(xy 254.635 102.87) (xy 254.635 99.06)
-		)
-		(stroke
-			(width 0)
-			(type default)
-		)
-	)
-	(wire
-		(pts
 			(xy 165.1 55.245) (xy 163.83 55.245)
 		)
@@
 	(wire
 		(pts
-			(xy 271.145 99.06) (xy 274.955 99.06)
+			(xy 270.51 99.06) (xy 274.955 99.06)
 		)
 		(stroke
@@
 		)
 	)
-	(wire
-		(pts
-			(xy 266.7 102.87) (xy 271.145 102.87)
-		)
-		(stroke
-			(width 0)
-			(type default)
-		)
-	)
 	(polyline
 		(pts
@@
 	(wire
 		(pts
-			(xy 251.46 99.06) (xy 254.635 99.06)
-		)
-		(stroke
-			(width 0)
-			(type default)
-		)
-	)
-	(wire
-		(pts
 			(xy 149.86 183.515) (xy 149.86 178.435)
 		)
@@
 	(wire
 		(pts
-			(xy 259.08 102.87) (xy 254.635 102.87)
-		)
-		(stroke
-			(width 0)
-			(type default)
-		)
-	)
-	(wire
-		(pts
 			(xy 45.72 93.98) (xy 43.18 93.98)
 		)
@@
 	(wire
 		(pts
-			(xy 270.51 99.06) (xy 271.145 99.06)
-		)
-		(stroke
-			(width 0)
-			(type default)
-		)
-	)
-	(wire
-		(pts
 			(xy 81.915 165.735) (xy 80.01 165.735)
 		)
@@
 					(unit 1)
 				)
-			)
-		)
-	)
-	(symbol
-		(lib_id "Device:C")
-		(at 262.89 102.87 270)
-		(unit 1)
-		(exclude_from_sim no)
-		(in_bom yes)
-		(on_board yes)
-		(dnp no)
-		(property "Reference" "C5"
-			(at 269.24 104.14 90)
-			(effects
-				(font
-					(size 1.27 1.27)
-				)
-			)
-		)
-		(property "Value" "100nF-Ceramic"
-			(at 269.24 101.6 90)
-			(effects
-				(font
-					(size 1.27 1.27)
-				)
-			)
-		)
-		(property "Footprint" "Capacitor_SMD:C_0402_1005Metric"
-			(at 259.08 103.8352 0)
-			(effects
-				(font
-					(size 1.27 1.27)
-				)
-				(hide yes)
-			)
-		)
-		(property "Datasheet" "~"
-			(at 262.89 102.87 0)
-			(effects
-				(font
-					(size 1.27 1.27)
-				)
-				(hide yes)
-			)
-		)
-		(property "Description" ""
-			(at 262.89 102.87 0)
-			(effects
-				(font
-					(size 1.27 1.27)
-				)
-				(hide yes)
-			)
-		)
-		(property "LCSC" "C1525"
-			(at 262.89 102.87 0)
-			(effects
-				(font
-					(size 1.27 1.27)
-				)
-				(hide yes)
-			)
-		)
-		(property "MPN" "C1525"
-			(at 262.89 102.87 0)
-			(effects
-				(font
-					(size 1.27 1.27)
-				)
-				(hide yes)
-			)
-		)
-		(property "JLCPCB Position Offset" ""
-			(at 262.89 102.87 0)
-			(effects
-				(font
-					(size 1.27 1.27)
-				)
-				(hide yes)
-			)
-		)
-		(pin "1"
-		)
-		(pin "2"
-		)
-		(instances
-			(project "Board"
-				(path "/fa2a81f8-bf39-4c28-beef-a6fc807c4564"
-					(reference "C5")
-					(unit 1)
-				)
